File: portal-gun/portal-gun.kicad_pcb (KiCad board)
At the start: 2 copper layers, 107.2 x 55.5 mm, 2 parts

Commit message: fast forward
Parts:
- removed the REF** at (146.2, 74.3)
- removed the REF** at (136.9, 88.7)
- added ?: , , F.Cu at (146.2, 74.2)
- added C1: C_Small, Capacitor_SMD:C_0603_1608Metric, B.Cu at (120.5, 79.7)
- added J1: SAO, Connector_PinHeader_2.54mm:PinHeader_2x03_P2.54mm_Vertical, B.Cu at (124.2, 87.3)
- added REF**: TestPoint_THTPad_D2.0mm_Drill1.0mm, TestPoint:TestPoint_THTPad_D2.0mm_Drill1.0mm, F.Cu at (136.9, 88.7)
- added SW1: SW_Push, Button_Switch_SMD:SW-SMD_GT-TC050C-H050-L1, B.Cu at (112.7, 85.5)
- added U1: ~, Package_TO_SOT_SMD:SOT-23-6, B.Cu at (120.5, 76.1)
- added U2: ~, LED_SMD:LED-SMD_5P-L3.2-W1.4_TX1813Y5, B.Cu at (128.6, 71.2)
- added U3: ~, LED_SMD:LED-SMD_5P-L3.2-W1.4_TX1813Y5, B.Cu at (152.1, 81.3)
- added U4: ~, LED_SMD:LED-SMD_5P-L3.2-W1.4_TX1813Y5, B.Cu at (160.9, 81.3)
- added U5: ~, LED_SMD:LED-SMD_5P-L3.2-W1.4_TX1813Y5, B.Cu at (195.7, 81.8)
Routing:
- net VDD: track 0.00 -> 128.8 mm
- net Net-(U4-DO): track 0.00 -> 35.5 mm
- net Net-(U2-DO): track 0.00 -> 30.8 mm
- net Net-(J1-Pin_5): track 0.00 -> 17.4 mm
- net Net-(J1-Pin_6): track 0.00 -> 15.8 mm
- net Net-(U1-PA4): track 0.00 -> 12.4 mm
- net Net-(U3-DO): track 0.00 -> 7.83 mm
- net Net-(U1-PA5): track 0.00 -> 7.18 mm
- net GND: track 0.00 -> 4.40 mm, vias 0 -> 6
- added copper zone on B.Cu, net GND
- added copper zone on F.Cu, net GND
- removed copper zone on F.Cu, net (none)
Other:
- board text added: "3.3v"
- board text added: "CK"
- board text added: "DA"
- board text added: "Gnd"
- board text added: "Portal Gun SAO www.BigFuckingBadge.com DC33"

Commit message: updated design with front fill as vcc
Parts:
- removed ?: , 
- added REF**: TestPoint_THTPad_D2.0mm_Drill1.0mm, TestPoint:TestPoint_THTPad_D2.0mm_Drill1.0mm, F.Cu at (146.2, 74.2)
Connections:
- SW1 pad 3: GND -> (no net)
- SW1 pad 4: GND -> (no net)
Routing:
- net VDD: track 128.8 -> 10.8 mm, vias 0 -> 6
- net Net-(U2-DO): track 30.8 -> 25.9 mm
- net GND: track 4.40 -> 0.00 mm, vias 6 -> 0
- net Net-(U4-DO): track 35.5 -> 34.9 mm
- added copper zone on F.Cu, net VDD
- removed copper zone on F.Cu, net GND
Other:
- board text added: "Abeth's Portal Gun SAO www.BigFuckingBadge.com DC33"
- board text removed: "Portal Gun SAO www.BigFuckingBadge.com DC33"
