File: portal-gun/portal-gun.kicad_pcb (KiCad board)
At the start: 2 copper layers, 107.2 x 55.5 mm, 10 parts, among them J1 SAO, SW1 SW_Push

Commit message: final proto updates
Parts:
- added REF**: MountingHole_2.1mm, MountingHole:MountingHole_2.1mm, F.Cu at (113.0, 77.3)
- added REF**: TestPoint_Pad_2.0x2.0mm, TestPoint:TestPoint_Pad_2.0x2.0mm, B.Cu at (171.8, 70.3)
- added REF**: TestPoint_Pad_2.0x2.0mm, TestPoint:TestPoint_Pad_2.0x2.0mm, B.Cu at (171.8, 94.6)
- renumbered SW1 to lanyard
Other:
- board text added: "3"
- board text added: "ABETH'S PORTAL GUN SAO"
- board text added: "DC3"
- board text added: "www.BigFuckingBadge.com"
- board text removed: "Abeth's Portal Gun SAO www.BigFuckingBadge.com DC33"
